File: Tamagotchi/Tamagotchi (mess up).kicad_pcb (KiCad board)
At the start: 2 copper layers, 8 parts, among them J1 Conn_01x20, J2 Conn_01x20, J4 Conn_01x07, J5 Conn_01x08, U1 TP4056-module

Commit message: tamagotchif older
Parts:
- moved J5 18.5 mm to (91.4, 152.4), turned to 180 degrees
- moved U1 17.8 mm to (109.2, 175.3)
Routing:
- net GND: track 112.8 -> 38.1 mm
- net +3.3V: track 123.6 -> 58.4 mm
- net Net-(U1-IN+): track 43.2 -> 0.00 mm
- net SDA: track 25.4 -> 5.08 mm
- net Net-(D1-A): track 25.4 -> 5.08 mm, vias 0 -> 1
- net INT1: track 17.8 -> 0.00 mm
- net SCL: track 15.2 -> 2.54 mm
