File: Tamagotchi/Tamagotchi.kicad_sch (KiCad schematic)
At the start: 4 parts, among them J1 Conn_01x20, J2 Conn_01x20, J3 Conn_01x06, J4 Conn_01x07

Commit message: schematic updated
Parts:
- added D1: 1N5817, Diode_THT:D_DO-41_SOD81_P10.16mm_Horizontal, symbol Diode:1N5817
- added J5: Conn_01x08, symbol Connector_Generic:Conn_01x08
- added R1: 680, symbol Device:R
- added R2: 1000, symbol Device:R
- added U1: TP4056-module, Package_SO:SOIC-8-1EP_3.9x4.9mm_P1.27mm_EP2.41x3.3mm_ThermalVias, symbol Tama_Symbols:TP4056-MODULE
Connections:
- net +3.3V: now also J2.16 (Pin_16), J4.6 (Pin_6), J5.2 (Pin_2), J5.6 (Pin_6); no longer J1.16 (Pin_16), J4.VCC (Pin_6)
- net GND: now also J2.18 (Pin_18), J4.7 (Pin_7), J5.1 (Pin_1), R2.2, U1. (OUT-); no longer J1.18 (Pin_18), J4.GND (Pin_7)
- net BAT: now reaches J2.19 (Pin_19)
- net BAT: now also D1.1 (K)
- net at J2.4 (Pin_4): no longer J4.CLK (Pin_5)
- net at J2.5 (Pin_5): no longer J4.MOSI (Pin_4)
- net at J2.6 (Pin_6): no longer J4.RES (Pin_3)
- net at J2.7 (Pin_7): no longer J4.DC (Pin_2)
- net at J2.9 (Pin_9): no longer J4.CS (Pin_1)
- net SDA: now reaches J1.1 (Pin_1)
- net SDA: now also J5.7 (Pin_7)
- net CHRG: now reaches J1.10 (Pin_10)
- net CHRG: now also R1.1, R2.1
- net INT1: now reaches J1.11 (Pin_11)
- net INT1: now also J5.4 (Pin_4)
- net SCL: now reaches J1.2 (Pin_2)
- net SCL: now also J5.8 (Pin_8)
- net CLK: now reaches J1.4 (Pin_4)
- net CLK: now also J4.5 (Pin_5)
- net MOSI: now reaches J1.5 (Pin_5)
- net MOSI: now also J4.4 (Pin_4)
- net RES: now reaches J1.6 (Pin_6)
- net RES: now also J4.3 (Pin_3)
- net DC: now reaches J1.7 (Pin_7)
- net DC: now also J4.2 (Pin_2)
- net CS: now reaches J1.9 (Pin_9)
- net CS: now also J4.1 (Pin_1), J5.3 (Pin_3)
- new net: D1.2 (A), U1. (OUT-)
- new net: R1.2, U1. (OUT-)
- new net +BATT: U1. (OUT-)
- new net -BATT: U1. (OUT-)
Other:
- note added: "ADXL345"
- note added: "usb"
- moved on the sheet: J4

Commit message: schematic updated
Parts:
- removed J3: Conn_01x06, symbol Connector_Generic:Conn_01x06
- J1, J2: footprint (none) -> Connector_PinHeader_2.54mm:PinHeader_1x20_P2.54mm_Vertical
- J4: footprint (none) -> Connector_PinHeader_2.54mm:Tama_Screen
- J5: footprint (none) -> Connector_PinHeader_2.54mm:Tama_Sensor
- R1, R2: footprint (none) -> Resistor_SMD:R_0201_0603Metric
- U1: footprint Package_SO:SOIC-8-1EP_3.9x4.9mm_P1.27mm_EP2.41x3.3mm_ThermalVias -> Connector_Hirose:Tama_TP4056
Connections:
- net +3.3V: now also J2.5 (Pin_5); no longer J2.16 (Pin_16)
- net +BATT: now also U1.4 (B+); no longer U1. (OUT-)
- net -BATT: now also U1.5 (B-); no longer U1. (OUT-)
- net BAT: now also J2.2 (Pin_2); no longer J2.19 (Pin_19)
- net CHRG: now also J2.19 (Pin_19); no longer J1.10 (Pin_10)
- net GND: now also J2.3 (Pin_3), U1.2 (IN-), U1.6 (OUT-); no longer J2.18 (Pin_18), U1. (OUT-)
- net at D1.2 (A): now also U1.3 (OUT+); no longer U1. (OUT-)
- net at R1.2: now also U1.1 (IN+); no longer U1. (OUT-)
Other:
- note removed: "sensor"
- moved on the sheet: J2
Changed lines of the file:
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@@
-		)
-	)
-	(text "sensor"
-		(exclude_from_sim no)
-		(at 191.008 61.976 0)
-		(effects
-			(font
-				(size 1.27 1.27)
-			)
 		)
 	)
@@
 	(wire
 		(pts
-			(xy 133.35 72.39) (xy 140.97 72.39)
+			(xy 130.81 72.39) (xy 140.97 72.39)
 		)
 		(stroke
@@
 	(wire
 		(pts
+			(xy 130.81 69.85) (xy 133.35 69.85)
+		)
+		(stroke
+			(width 0)
+			(type default)
+		)
+	)
+	(wire
+		(pts
 			(xy 140.97 69.85) (xy 143.51 69.85)
 		)
@@
 	(wire
 		(pts
+			(xy 130.81 77.47) (xy 147.32 77.47)
+		)
+		(stroke
+			(width 0)
+			(type default)
+		)
+	)
+	(wire
+		(pts
 			(xy 139.7 110.49) (xy 149.86 110.49)
 		)
@@
 		(pts
 			(xy 167.64 78.74) (xy 172.72 78.74)
-		)
-		(stroke
-			(width 0)
-			(type default)
-		)
-	)
-	(wire
-		(pts
-			(xy 133.35 77.47) (xy 147.32 77.47)
 		)
 		(stroke
@@
 	(global_label "CHRG"
 		(shape input)
-		(at 111.76 90.17 180)
-		(fields_autoplaced yes)
-		(effects
-			(font
-				(size 1.27 1.27)
-			)
-			(justify right)
+		(at 130.81 113.03 0)
+		(fields_autoplaced yes)
+		(effects
+			(font
+				(size 1.27 1.27)
+			)
+			(justify left)
 		)
 		(property "Intersheetrefs" "${INTERSHEET_REFS}"
-			(at 103.6343 90.17 0)
-			(effects
-				(font
-					(size 1.27 1.27)
-				)
-				(justify right)
+			(at 138.9357 113.03 0)
+			(effects
+				(font
+					(size 1.27 1.27)
+				)
+				(justify left)
 				(hide yes)
 			)
@@
 	(symbol
 		(lib_id "Connector_Generic:Conn_01x20")
-		(at 128.27 92.71 180)
+		(at 125.73 90.17 0)
+		(mirror y)
 		(unit 1)
 		(exclude_from_sim no)
@@
 		(on_board yes)
 		(dnp no)
-		(fields_autoplaced yes)
 		(property "Reference" "J2"
-			(at 128.27 60.96 0)
+			(at 125.73 121.92 0)
 			(effects
 				(font
@@
 		)
 		(property "Value" "Conn_01x20"
-			(at 128.27 63.5 0)
-			(effects
-				(font
-					(size 1.27 1.27)
-				)
-			)
-		)
-		(property "Footprint" ""
-			(at 128.27 92.71 0)
+			(at 125.73 119.38 0)
+			(effects
+				(font
+					(size 1.27 1.27)
+				)
+			)
+		)
+		(property "Footprint" "Connector_PinHeader_2.54mm:PinHeader_1x20_P2.54mm_Vertical"
+			(at 125.73 90.17 0)
 			(effects
 				(font
@@
 		)
 		(property "Datasheet" "~"
-			(at 128.27 92.71 0)
+			(at 125.73 90.17 0)
 			(effects
 				(font
@@
 		)
 		(property "Description" "Generic connector, single row, 01x20, script generated (kicad-library-utils/schlib/autogen/connector/)"
-			(at 128.27 92.71 0)
+			(at 125.73 90.17 0)
 			(effects
 				(font
@@
 			)
 		)
-		(property "Footprint" ""
+		(property "Footprint" "Connector_PinHeader_2.54mm:Tama_Screen"
 			(at 154.94 105.41 0)
 			(effects
@@
 			)
 		)
-		(property "Footprint" ""
+		(property "Footprint" "Connector_PinHeader_2.54mm:PinHeader_1x20_P2.54mm_Vertical"
 			(at 116.84 90.17 0)
 			(effects
@@
 				(path "/946c8241-5864-4868-8182-a8df1a8961a2"
 					(reference "J1")
-					(unit 1)
-				)
-			)
-		)
-	)
-	(symbol
-		(lib_id "Connector_Generic:Conn_01x06")
-		(at 175.26 67.31 0)
-		(unit 1)
-		(exclude_from_sim no)
-		(in_bom yes)
-		(on_board yes)
-		(dnp no)
-		(fields_autoplaced yes)
-		(property "Reference" "J3"
-			(at 177.8 67.3099 0)
-			(effects
-				(font
-					(size 1.27 1.27)
-				)
-				(justify left)
-			)
-		)
-		(property "Value" "Conn_01x06"
-			(at 177.8 69.8499 0)
-			(effects
-				(font
-					(size 1.27 1.27)
-				)
-				(justify left)
-			)
-		)
-		(property "Footprint" ""
-			(at 175.26 67.31 0)
-			(effects
-				(font
-					(size 1.27 1.27)
-				)
-				(hide yes)
-			)
-		)
-		(property "Datasheet" "~"
-			(at 175.26 67.31 0)
-			(effects
-				(font
-					(size 1.27 1.27)
-				)
-				(hide yes)
-			)
-		)
-		(property "Description" "Generic connector, single row, 01x06, script generated (kicad-library-utils/schlib/autogen/connector/)"
-			(at 175.26 67.31 0)
-			(effects
-				(font
-					(size 1.27 1.27)
-				)
-				(hide yes)
-			)
-		)
-		(pin "4"
-		)
-		(pin "5"
-		)
-		(pin "6"
-		)
-		(pin "3"
-		)
-		(pin "1"
-		)
-		(pin "2"
-		)
-		(instances
-			(project ""
-				(path "/946c8241-5864-4868-8182-a8df1a8961a2"
-					(reference "J3")
 					(unit 1)
 				)
@@
 		(on_board yes)
 		(dnp no)
-		(fields_autoplaced yes)
 		(property "Reference" "J5"
-			(at 182.88 87.6299 0)
+			(at 182.88 87.63 0)
 			(effects
 				(font
@@
 			)
 		)
-		(property "Footprint" ""
+		(property "Footprint" "Connector_PinHeader_2.54mm:Tama_Sensor"
 			(at 180.34 87.63 0)
 			(effects
@@
 			)
 		)
-		(property "Footprint" ""
+		(property "Footprint" "Resistor_SMD:R_0201_0603Metric"
 			(at 127 34.798 90)
 			(effects
@@
 			)
 		)
-		(property "Footprint" ""
+		(property "Footprint" "Resistor_SMD:R_0201_0603Metric"
 			(at 127 48.768 90)
 			(effects
@@
 			)
 		)
-		(property "Footprint" "Package_SO:SOIC-8-1EP_3.9x4.9mm_P1.27mm_EP2.41x3.3mm_ThermalVias"
+		(property "Footprint" "Connector_Hirose:Tama_TP4056"
 			(at 149.098 62.23 0)
 			(effects
@@
 			)
 		)
-		(pin ""
-		)
-		(pin ""
-		)
-		(pin ""
-		)
-		(pin ""
-		)
-		(pin ""
-		)
-		(pin ""
+		(pin "2"
+		)
+		(pin "3"
+		)
+		(pin "1"
+		)
+		(pin "5"
+		)
+		(pin "6"
+		)
+		(pin "4"
 		)
 		(instances

Commit message: tamagotchif older
Parts:
- D1: footprint Diode_THT:D_DO-41_SOD81_P10.16mm_Horizontal -> Diode_THT:D_DO-41_SOD81_P7.62mm_Horizontal
- R1, R2: footprint Resistor_SMD:R_0201_0603Metric -> Diode_THT:D_A-405_P7.62mm_Horizontal
Connections:
- net +3.3V: now also J5.3 (Pin_3)
- net CHRG: now also J1.15 (Pin_15); no longer J2.19 (Pin_19)
- net CS: now also J1.11 (Pin_11); no longer J1.9 (Pin_9), J5.3 (Pin_3)
- net DC: now also J1.10 (Pin_10); no longer J1.7 (Pin_7)
- net GND: now also J1.3 (Pin_3), J1.8 (Pin_8)
- net INT1: now also J1.20 (Pin_20); no longer J1.11 (Pin_11)
- net RES: now also J1.9 (Pin_9); no longer J1.6 (Pin_6)
- net SCL: now also J1.17 (Pin_17); no longer J1.2 (Pin_2)
- net SDA: now also J1.16 (Pin_16); no longer J1.1 (Pin_1)
